File: clap_on_off_switch.kicad_pcb (KiCad board)
At the start: 2 copper layers, 58.2 x 42.8 mm, 34 parts, among them J1 AC Switched Out, J2 220V AC IN, K1 relay_spst, Q1 MMBT2222A, U1 LM358, U2 NE556, U3 74HC08, U4 4013, U5 AC-DC_Converter

Commit message: README.md modified
Other:
- board text added: "Clap on/off switch v1.2"
- board text removed: "Clap on/off switch v1.1"
Changed lines of the file:
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@@
 		)
 	)
-	(gr_text "Clap on/off switch v1.1"
+	(gr_text "Clap on/off switch v1.2"
 		(at 157.8 76.15 0)
 		(layer "F.SilkS")
