File: clap_on_off_switch.kicad_sch (KiCad schematic)
At the start: 34 parts, among them J1 AC Switched Out, J2 220V AC IN, K1 relay_spst, Q1 MMBT2222A, U1 LM358, U2 NE556, U3 74HC08, U4 4013, U5 AC-DC_Converter

Commit message: README.md modified
Other:
- moved on the sheet: C1, MK1, R1, R4, R5, R6, R7, RV1, U1A, U1B
